File: Hardware/SE-VGA.kicad_pcb (KiCad board)
At the start: 2 copper layers, 101.6 x 101.6 mm, 78 parts, among them J1 PGM, J2 650946-5, J3 DE15_Receptacle_HighDensity_M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, J4 Conn_02x05_Odd_Even, J5 Conn_02x05_Odd_Even, SW1 SW_DIP_x06, U1 68000-CPU, U10 74HCT125D, U11 APX803S00-29SA-7, U14 AZ1117IH-1.2TRG1, U15 AZ1117IH-3.3TRG1, U2 SN74LVCH16T245, U3 SN74LVCH16T245, U4 SN74LVCH16T245, U5 IS42S16100H, U6 W25Q80DVSNIG, U7 ADA4891-4, U8 ICE40HX4K-TQ144, U9 68000-BOARD, X1 ECS-2333-100-BN-TR

Commit message: R3 PCB layout first draft
Parts:
- added C24: 1uF, Capacitor_SMD:C_0805_2012Metric_Pad1.18x1.45mm_HandSolder, F.Cu at (240.0, 106.7)
- added C25: 4.7uF, Capacitor_SMD:C_0805_2012Metric_Pad1.18x1.45mm_HandSolder, F.Cu at (263.5, 141.6)
- added C26: 4.7uF, Capacitor_SMD:C_0805_2012Metric_Pad1.18x1.45mm_HandSolder, F.Cu at (210.2, 140.3)
- added C27: 1uF, Capacitor_SMD:C_0805_2012Metric_Pad1.18x1.45mm_HandSolder, F.Cu at (210.2, 137.8)
- added C28: 1uF, Capacitor_SMD:C_0805_2012Metric_Pad1.18x1.45mm_HandSolder, F.Cu at (206.4, 137.8)
- added C34: 4.7uF, Capacitor_SMD:C_0805_2012Metric_Pad1.18x1.45mm_HandSolder, F.Cu at (206.4, 140.3)
- added REF**: MouseBite, SE-VGA:MouseBite, F.Cu at (201.9, 147.3)
- added REF**: MouseBite, SE-VGA:MouseBite, F.Cu at (201.9, 97.8)
- added REF**: MouseBite, SE-VGA:MouseBite, F.Cu at (201.9, 196.8)
- J5: moved to B.Cu
- moved C6 141.8 mm to (279.4, 121.3), turned to 180 degrees
- moved C14 132.1 mm to (261.0, 141.6), turned to 90 degrees
- moved C11 131.8 mm to (259.7, 133.3), turned to 180 degrees
- moved J3 131.6 mm to (189.9, 152.0), turned to -90 degrees
- moved C8 130.2 mm to (251.5, 140.2), turned to 180 degrees
- moved C3 130.0 mm to (259.1, 127.6), turned to 90 degrees
- moved C4 130.0 mm to (261.6, 127.6), turned to 90 degrees
- moved C15 128.2 mm to (258.4, 141.6), turned to 90 degrees
- moved C5 123.5 mm to (266.7, 112.4), turned to -90 degrees
- moved C18 123.3 mm to (282.6, 103.5), turned to 90 degrees
- moved R14 121.8 mm to (292.1, 112.4), turned to -90 degrees
- moved C7 120.7 mm to (232.4, 139.7)
- moved R15 118.3 mm to (289.6, 112.4), turned to -90 degrees
- moved R16 117.4 mm to (287.0, 112.4), turned to -90 degrees
- moved R6 114.2 mm to (283.2, 94.0), turned to 180 degrees
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Connections:
- C14 pad 2: +3V3 -> +1V2
- R13 pad 2: Net-(U7D-OUT4) -> Net-(U7B-OUT2)
- R2 pad 1: Net-(U7B-IN2_N) -> Net-(U7D-IN4_N)
- U7 pad 12: +5V -> Net-(RN4B-R2.2)
- U7 pad 13: +5V -> Net-(U7D-IN4_N)
- U7 pad 14: Net-(U7D-OUT4) -> Net-(U7D-IN4_N)
- U7 pad 5: Net-(RN4B-R2.2) -> +5V
- U7 pad 6: Net-(U7B-IN2_N) -> +5V
- U7 pad 7: Net-(U7B-IN2_N) -> Net-(U7B-OUT2)
- U8 pad 101: /VRAM-A4 -> /VRAM-D12
- U8 pad 102: /VRAM-A5 -> /VRAM-D11
- U8 pad 104: /VRAM-A6 -> /VRAM-D10
- U8 pad 105: /VRAM-A7 -> /VRAM-D9
- U8 pad 106: /VRAM-A8 -> /VRAM-D8
- U8 pad 107: /VRAM-A9 -> /VRAM-UDQM
- U8 pad 110: unconnected-(U8A-IOT_168-Pad110) -> /VRAM-CLK
- U8 pad 112: unconnected-(U8A-IOT_169-Pad112) -> /VRAM-CKE
- U8 pad 113: unconnected-(U8A-IOT_170-Pad113) -> /VRAM-A9
- U8 pad 114: unconnected-(U8A-IOT_171-Pad114) -> /VRAM-A8
- U8 pad 115: unconnected-(U8A-IOT_172-Pad115) -> /VRAM-A7
- U8 pad 116: unconnected-(U8A-IOT_173-Pad116) -> /VRAM-A6
- U8 pad 117: unconnected-(U8A-IOT_174-Pad117) -> /VRAM-A5
- U8 pad 118: unconnected-(U8A-IOT_177-Pad118) -> /VRAM-A4
- U8 pad 119: unconnected-(U8A-IOT_178-Pad119) -> /VRAM-D0
- U8 pad 120: unconnected-(U8A-IOT_179-Pad120) -> /VRAM-D1
- U8 pad 121: unconnected-(U8A-IOT_181-Pad121) -> /VRAM-D2
- U8 pad 122: unconnected-(U8A-IOT_190-Pad122) -> /VRAM-D3
- U8 pad 124: unconnected-(U8A-IOT_191-Pad124) -> /VRAM-D4
- U8 pad 125: unconnected-(U8A-IOT_192-Pad125) -> /VRAM-D5
- U8 pad 128: unconnected-(U8A-IOT_197_GBIN1-Pad128) -> /VRAM-D6
- U8 pad 129: unconnected-(U8A-IOT_198_GBIN0-Pad129) -> /VRAM-D7
- U8 pad 130: unconnected-(U8A-IOT_206-Pad130) -> /VRAM-LDQM
- U8 pad 134: unconnected-(U8A-IOT_212-Pad134) -> /~{VRAM-WE}
- U8 pad 135: unconnected-(U8A-IOT_213-Pad135) -> /~{VRAM-CAS}
- U8 pad 136: unconnected-(U8A-IOT_214-Pad136) -> /~{VRAM-RAS}
- U8 pad 137: unconnected-(U8A-IOT_215-Pad137) -> /~{VRAM-CS}
- U8 pad 138: unconnected-(U8A-IOT_216-Pad138) -> /VRAM-A1
- U8 pad 139: unconnected-(U8A-IOT_217-Pad139) -> /VRAM-A2
- U8 pad 141: unconnected-(U8A-IOT_219-Pad141) -> /VRAM-A11
- U8 pad 142: unconnected-(U8A-IOT_220-Pad142) -> /VRAM-A10
- U8 pad 143: unconnected-(U8A-IOT_221-Pad143) -> /VRAM-A0
- U8 pad 144: unconnected-(U8A-IOT_222-Pad144) -> /VRAM-A3
- U8 pad 73: unconnected-(U8B-IOR_109-Pad73) -> /VID-B2
- U8 pad 74: unconnected-(U8B-IOR_110-Pad74) -> /VID-B3
- U8 pad 75: unconnected-(U8B-IOR_111-Pad75) -> /VID-B0
- U8 pad 76: unconnected-(U8B-IOR_112-Pad76) -> /VID-VSYNC3
- U8 pad 78: unconnected-(U8B-IOR_114-Pad78) -> /VID-HSYNC3
- U8 pad 79: unconnected-(U8B-IOR_115-Pad79) -> /VID-B1
- U8 pad 80: unconnected-(U8B-IOR_116-Pad80) -> /VID-G2
- U8 pad 81: unconnected-(U8B-IOR_117-Pad81) -> /VID-G3
- U8 pad 82: unconnected-(U8B-IOR_118-Pad82) -> /VID-G0
- U8 pad 83: unconnected-(U8B-IOR_119-Pad83) -> /VID-G1
- U8 pad 84: unconnected-(U8B-IOR_120-Pad84) -> /VID-R2
- U8 pad 85: unconnected-(U8B-IOR_128-Pad85) -> /VID-R3
- U8 pad 87: unconnected-(U8B-IOR_136-Pad87) -> /VID-R0
- U8 pad 88: unconnected-(U8B-IOR_137-Pad88) -> /VID-R1
- U8 pad 91: unconnected-(U8B-IOR_139-Pad91) -> /AUXSW
- U8 pad 94: /VRAM-UDQM -> /MEMSEL0
- U8 pad 95: unconnected-(U8B-IOR_144-Pad95) -> /MEMSEL1
- U8 pad 96: unconnected-(U8B-IOR_146-Pad96) -> /MEMSEL2
- U8 pad 97: unconnected-(U8B-IOR_147-Pad97) -> /VRAM-D15
- U8 pad 98: /VRAM-A2 -> /VRAM-D14
- U8 pad 99: /VRAM-A3 -> /VRAM-D13
Routing:
- net +3V3: track 3.30 -> 410.7 mm, vias 0 -> 46
- net +5V: track 0.00 -> 206.3 mm, vias 0 -> 25
- net GND: track 0.00 -> 183.7 mm, vias 0 -> 167
- net /VID-VSYNC: track 0.00 -> 177.3 mm
- net /VID-HSYNC: track 0.00 -> 172.7 mm
- net +1V2: track 3.30 -> 138.1 mm, vias 0 -> 28
- net /AUXSW: track 0.00 -> 107.7 mm, vias 0 -> 1
- net /MEMSEL2: track 0.00 -> 100.9 mm, vias 0 -> 1
- net /MEMSEL1: track 0.00 -> 96.8 mm, vias 0 -> 1
- net /MEMSEL0: track 0.00 -> 95.2 mm, vias 0 -> 1
- net /VID-R-A: track 0.00 -> 81.5 mm
- net /VID-B-A: track 0.00 -> 81.3 mm
- net /VID-G-A: track 0.00 -> 80.8 mm
- net /~{CPU-DTACK}: track 58.2 -> 124.8 mm, vias 3 -> 2
- net /VID-HSYNC3: track 0.00 -> 53.9 mm
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- added copper zone on B.Cu, net +1V2
- added copper zone on F.Cu, net +1V2
- added copper zone on B.Cu, net +3V3
- added copper zone on F.Cu, net +3V3
- added copper zone on B.Cu, net GND
- added copper zone on F.Cu, net GND
Other:
- board size 101.6 x 101.6 mm -> 127.6 x 114.3 mm
- board text added: "SE"
- board text added: "VGA"
- board text added: "techav"
