File: Hardware/SE-VGA.kicad_sch (KiCad schematic)
At the start: 67 parts, among them J1 PGM, J3 DE15_Receptacle_HighDensity_M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, J4 Conn_02x05_Odd_Even, J5 Conn_02x05_Odd_Even, SW1 SW_DIP_x06, U10 74HCT125D, U11 APX803S00-29SA-7, U12 AZ1117IH-1.2TRG1, U13 AZ1117IH-3.3TRG1, U5 IS42S16100H, U6 W25Q80DVSNIG, U7 ADA4891-4, U8 ICE40HX4K-TQ144, X1 ECS-2333-100-BN-TR

Commit message: R3 Initial schematic complete, start routing
Connections:
- net +5V: now also U10.1; no longer U10.13
- net AUXSW: no longer U8.34 (IOL_25B)
- net CPU3-A1: now also U8.9 (IOL_5A); no longer U8.115 (IOT_172)
- net CPU3-A10: now also U8.12 (IOL_8B); no longer U8.125 (IOT_192)
- net CPU3-A11: now also U8.15 (IOL_10A); no longer U8.128 (IOT_197_GBIN1)
- net CPU3-A12: now also U8.16 (IOL_10B); no longer U8.129 (IOT_198_GBIN0)
- net CPU3-A13: now also U8.18 (IOL_12B); no longer U8.130 (IOT_206)
- net CPU3-A14: now also U8.17 (IOL_12A); no longer U8.134 (IOT_212)
- net CPU3-A15: now also U8.19 (IOL_13A); no longer U8.135 (IOT_213)
- net CPU3-A16: now also U8.20 (IOL_13B_GBIN7); no longer U8.136 (IOT_214)
- net CPU3-A17: now also U8.21 (IOL_14A_GBIN6); no longer U8.137 (IOT_215)
- net CPU3-A18: now also U8.22 (IOL_14B); no longer U8.138 (IOT_216)
- net CPU3-A19: now also U8.23 (IOL_17A); no longer U8.139 (IOT_217)
- net CPU3-A2: now also U8.7 (IOL_4A); no longer U8.116 (IOT_173)
- net CPU3-A20: now also U8.24 (IOL_17B); no longer U8.141 (IOT_219)
- net CPU3-A21: now also U8.25 (IOL_18A); no longer U8.142 (IOT_220)
- net CPU3-A22: now also U8.26 (IOL_18B); no longer U8.143 (IOT_221)
- net CPU3-A23: now also U8.28 (IOL_23A); no longer U8.144 (IOT_222)
- net CPU3-A3: now also U8.3 (IOL_3A); no longer U8.117 (IOT_174)
- net CPU3-A4: now also U8.1 (IOL_2A); no longer U8.118 (IOT_177)
- net CPU3-A5: now also U8.2 (IOL_2B); no longer U8.119 (IOT_178)
- net CPU3-A6: now also U8.4 (IOL_3B); no longer U8.120 (IOT_179)
- net CPU3-A7: now also U8.8 (IOL_4B); no longer U8.121 (IOT_181)
- net CPU3-A8: now also U8.10 (IOL_5B); no longer U8.122 (IOT_190)
- net CPU3-A9: now also U8.11 (IOL_8A); no longer U8.124 (IOT_191)
- net CPU3-D0: now also U8.47 (IOB_79); no longer U8.73 (IOR_109)
- net CPU3-D1: now also U8.49 (IOB_81_GBIN5); no longer U8.74 (IOR_110)
- net CPU3-D10: now also U8.44 (IOB_72); no longer U8.84 (IOR_120)
- net CPU3-D11: now also U8.43 (IOB_71); no longer U8.85 (IOR_128)
- net CPU3-D12: now also U8.42 (IOB_64); no longer U8.87 (IOR_136)
- net CPU3-D13: now also U8.41 (IOB_63); no longer U8.88 (IOR_137)
- net CPU3-D14: now also U8.39 (IOB_61); no longer U8.90 (IOR_138)
- net CPU3-D15: now also U8.38 (IOB_57); no longer U8.91 (IOR_139)
- net CPU3-D2: now also U8.55 (IOB_91); no longer U8.75 (IOR_111)
- net CPU3-D3: now also U8.56 (IOB_94); no longer U8.76 (IOR_112)
- net CPU3-D4: now also U8.62 (IOB_102); no longer U8.78 (IOR_114)
- net CPU3-D5: now also U8.61 (IOB_96); no longer U8.79 (IOR_115)
- net CPU3-D6: now also U8.60 (IOB_95); no longer U8.80 (IOR_116)
- net CPU3-D7: now also U8.52 (IOB_82_GBIN4); no longer U8.81 (IOR_117)
- net CPU3-D8: now also U8.48 (IOB_80); no longer U8.82 (IOR_118)
- net CPU3-D9: now also U8.45 (IOB_73); no longer U8.83 (IOR_119)
- net CPU3-R/~{W}: now also U8.29 (IOL_23B); no longer U8.62 (IOB_102)
- net GND: now also U10.10, U10.13, U10.2, U10.3, U10.5; no longer U10.1, U10.11, U10.12, U10.4, U10.9
- net MEMSEL0: no longer U8.25 (IOL_18A)
- net MEMSEL1: no longer U8.26 (IOL_18B)
- net MEMSEL2: no longer U8.28 (IOL_23A)
- net VID-B0: no longer U8.11 (IOL_8A)
- net VID-B1: no longer U8.12 (IOL_8B)
- net VID-B2: no longer U8.15 (IOL_10A)
- net VID-B3: no longer U8.16 (IOL_10B)
- net VID-G0: no longer U8.7 (IOL_4A)
- net VID-G1: no longer U8.8 (IOL_4B)
- net VID-G2: no longer U8.9 (IOL_5A)
- net VID-G3: no longer U8.10 (IOL_5B)
- net VID-HSYNC: now also U10.8; no longer U10.3
- net VID-HSYNC3: now also U10.9; no longer U10.2, U8.17 (IOL_12A)
- net VID-R0: no longer U8.1 (IOL_2A)
- net VID-R1: no longer U8.2 (IOL_2B)
- net VID-R2: no longer U8.3 (IOL_3A)
- net VID-R3: no longer U8.4 (IOL_3B)
- net VID-VSYNC: now also U10.11; no longer U10.6
- net VID-VSYNC3: now also U10.12; no longer U10.5, U8.18 (IOL_12B)
- net VRAM-A0: no longer U8.96 (IOR_146)
- net VRAM-A1: no longer U8.97 (IOR_147)
- net VRAM-A10: no longer U8.110 (IOT_168)
- net VRAM-A11: no longer U8.112 (IOT_169)
- net VRAM-CKE: no longer U8.24 (IOL_17B)
- net VRAM-CLK: no longer U8.23 (IOL_17A)
- net VRAM-D0: no longer U8.37 (IOB_56)
- net VRAM-D1: no longer U8.38 (IOB_57)
- net VRAM-D10: no longer U8.49 (IOB_81_GBIN5)
- net VRAM-D11: no longer U8.52 (IOB_82_GBIN4)
- net VRAM-D12: no longer U8.55 (IOB_91)
- net VRAM-D13: no longer U8.56 (IOB_94)
- net VRAM-D14: no longer U8.60 (IOB_95)
- net VRAM-D15: no longer U8.61 (IOB_96)
- net VRAM-D2: no longer U8.39 (IOB_61)
- net VRAM-D3: no longer U8.41 (IOB_63)
- net VRAM-D4: no longer U8.42 (IOB_64)
- net VRAM-D5: no longer U8.43 (IOB_71)
- net VRAM-D6: no longer U8.44 (IOB_72)
- net VRAM-D7: no longer U8.45 (IOB_73)
- net VRAM-D8: no longer U8.47 (IOB_79)
- net VRAM-D9: no longer U8.48 (IOB_80)
- net VRAM-LDQM: no longer U8.95 (IOR_144)
- net ~{CPU-DTACK}: now also U10.6; no longer U10.8
- net ~{CPU3-AS}: now also U8.33 (IOL_25A); no longer U8.113 (IOT_170)
- net ~{CPU3-DEN}: now also U8.37 (IOB_56); no longer U8.29 (IOL_23B)
- net ~{CPU3-DTACK}: now also U10.4, U8.34 (IOL_25B); no longer U10.10, U8.33 (IOL_25A)
- net ~{CPU3-LDS}: now also U8.31 (IOL_24A); no longer U8.32 (IOL_24B)
- net ~{CPU3-UDS}: now also U8.32 (IOL_24B); no longer U8.31 (IOL_24A)
- net ~{VRAM-CAS}: no longer U8.19 (IOL_13A)
- net ~{VRAM-CS}: no longer U8.22 (IOL_14B)
- net ~{VRAM-RAS}: no longer U8.20 (IOL_13B_GBIN7)
- net ~{VRAM-WE}: no longer U8.21 (IOL_14A_GBIN6)
- net CPU3-A0: no longer names the net of U8.114 (IOT_171)
Other:
- moved on the sheet: U10A, U10B, U10C, U10D, U8D

Commit message: R3 PCB layout first draft
Parts:
- added C24, C27, C28: 1uF, Capacitor_SMD:C_0805_2012Metric_Pad1.18x1.45mm_HandSolder, symbol Device:C_Small
- added C25, C26, C34: 4.7uF, Capacitor_SMD:C_0805_2012Metric_Pad1.18x1.45mm_HandSolder, symbol Device:C_Small
Connections:
- net +1V2: now also C14.2, C25.2
- net +3V3: now also C24.1, C26.2, C27.2, C28.2, C34.2; no longer C14.2
- net +5V: now also U7.5 (IN2_P), U7.6 (IN2_N); no longer U7.12 (IN4_P), U7.13 (IN4_N)
- net AUXSW: now also U8.91 (IOR_139)
- net GND: now also C24.2, C25.1, C26.1, C27.1, C28.1, C34.1
- net MEMSEL0: now also U8.94 (IOR_141_GBIN2)
- net MEMSEL1: now also U8.95 (IOR_144)
- net MEMSEL2: now also U8.96 (IOR_146)
- net VID-B0: now also U8.75 (IOR_111)
- net VID-B1: now also U8.79 (IOR_115)
- net VID-B2: now also U8.73 (IOR_109)
- net VID-B3: now also U8.74 (IOR_110)
- net VID-G0: now also U8.82 (IOR_118)
- net VID-G1: now also U8.83 (IOR_119)
- net VID-G2: now also U8.80 (IOR_116)
- net VID-G3: now also U8.81 (IOR_117)
- net VID-HSYNC3: now also U8.78 (IOR_114)
- net VID-R0: now also U8.87 (IOR_136)
- net VID-R1: now also U8.88 (IOR_137)
- net VID-R2: now also U8.84 (IOR_120)
- net VID-R3: now also U8.85 (IOR_128)
- net VID-VSYNC3: now also U8.76 (IOR_112)
- net VRAM-A0: now also U8.143 (IOT_221)
- net VRAM-A1: now also U8.138 (IOT_216)
- net VRAM-A10: now also U8.142 (IOT_220)
- net VRAM-A11: now also U8.141 (IOT_219)
- net VRAM-A2: now also U8.139 (IOT_217); no longer U8.98 (IOR_148)
- net VRAM-A3: now also U8.144 (IOT_222); no longer U8.99 (IOR_152)
- net VRAM-A4: now also U8.118 (IOT_177); no longer U8.101 (IOR_160)
- net VRAM-A5: now also U8.117 (IOT_174); no longer U8.102 (IOR_161)
- net VRAM-A6: now also U8.116 (IOT_173); no longer U8.104 (IOR_164)
- net VRAM-A7: now also U8.115 (IOT_172); no longer U8.105 (IOR_165)
- net VRAM-A8: now also U8.114 (IOT_171); no longer U8.106 (IOR_166)
- net VRAM-A9: now also U8.113 (IOT_170); no longer U8.107 (IOR_167)
- net VRAM-CKE: now also U8.112 (IOT_169)
- net VRAM-CLK: now also U8.110 (IOT_168)
- net VRAM-D0: now also U8.119 (IOT_178)
- net VRAM-D1: now also U8.120 (IOT_179)
- net VRAM-D10: now also U8.104 (IOR_164)
- net VRAM-D11: now also U8.102 (IOR_161)
- net VRAM-D12: now also U8.101 (IOR_160)
- net VRAM-D13: now also U8.99 (IOR_152)
- net VRAM-D14: now also U8.98 (IOR_148)
- net VRAM-D15: now also U8.97 (IOR_147)
- net VRAM-D2: now also U8.121 (IOT_181)
- net VRAM-D3: now also U8.122 (IOT_190)
- net VRAM-D4: now also U8.124 (IOT_191)
- net VRAM-D5: now also U8.125 (IOT_192)
- net VRAM-D6: now also U8.128 (IOT_197_GBIN1)
- net VRAM-D7: now also U8.129 (IOT_198_GBIN0)
- net VRAM-D8: now also U8.106 (IOR_166)
- net VRAM-D9: now also U8.105 (IOR_165)
- net VRAM-LDQM: now also U8.130 (IOT_206)
- net VRAM-UDQM: now also U8.107 (IOR_167); no longer U8.94 (IOR_141_GBIN2)
- net ~{VRAM-CAS}: now also U8.135 (IOT_213)
- net ~{VRAM-CS}: now also U8.137 (IOT_215)
- net ~{VRAM-RAS}: now also U8.136 (IOT_214)
- net ~{VRAM-WE}: now also U8.134 (IOT_212)
- net at R5.2, RN4.7 (R2.2), RN6.1 (R1.1): now also U7.12 (IN4_P); no longer U7.5 (IN2_P)
- net at R13.2: now also U7.7 (OUT2); no longer U7.14 (OUT4)
- new net: R2.1, U7.13 (IN4_N), U7.14 (OUT4)
Other:
- moved on the sheet: C10, C14, C7, C8, C9, U7B, U7D

Commit message: Multiplex CPU bus and add 24bpp output
Parts:
- removed J3: DE15_Receptacle_HighDensity_MountingHoles, Connector_Dsub:DSUB-15-HD_Female_Vertical_P2.29x1.98mm_MountingHoles, symbol Connector:DE15_Receptacle_HighDensity_MountingHoles
- removed J5: Conn_02x05_Odd_Even, Connector_PinHeader_2.54mm:PinHeader_2x05_P2.54mm_Vertical, symbol Connector_Generic:Conn_02x05_Odd_Even
- removed RN1, RN10, RN2, RN3, RN4, RN5, RN6, RN7, RN8, RN9: CAY16-1500F4LF, Resistor_SMD:R_Array_Convex_4x1206, symbol Device:R_Pack04_Split
- removed U5: IS42S16100H, SE-VGA:TSOP2-50, symbol SE-VGA:IS42S16100H
- added R21, R22, R23, R24, R25, R26, R27, R28, R29, R37, R38, R39, R40, R41, R42, R43, R44, R52, R53, R54, R55, R56, R57, R58, R59, R60, R68: 300R, Resistor_SMD:R_0402_1005Metric, symbol Device:R_Small_US
- added R30, R31, R32, R33, R34, R35, R36, R45, R46, R47, R48, R49, R50, R51, R61, R62, R63, R64, R65, R66, R67: 150R, Resistor_SMD:R_0402_1005Metric, symbol Device:R_Small_US
- added U12: MT48LC16M16A2P, Package_SO:TSOP-II-54_22.2x10.16mm_P0.8mm, symbol Memory_RAM:MT48LC16M16A2P
- C1, C10, C11, C12, C13, C14, C15, C16, C17, C18, C2, C24, C25, C26, C27, C28, C3, C32, C33, C34, C4, C5, C6, C7, C8, C9: footprint Capacitor_SMD:C_0805_2012Metric_Pad1.18x1.45mm_HandSolder -> Capacitor_SMD:C_0402_1005Metric
- R1, R10, R11, R12, R13, R14, R15, R16, R17, R18, R19, R2, R20, R3, R4, R5, R6, R7, R8, R9: footprint Resistor_SMD:R_0805_2012Metric_Pad1.20x1.40mm_HandSolder -> Resistor_SMD:R_0402_1005Metric
- renumbered J4 to J3, U12 to U14, U13 to U15
Connections:
- net CPU3-A1 is gone; now on net CPU3-A21: U8.9 (IOL_5A)
- net CPU3-A10 is gone; now on net CPU3-A18: U8.12 (IOL_8B)
- net CPU3-A11 is gone; now on net CPU3-A17: U8.15 (IOL_10A)
- net CPU3-A12 is gone; now on net CPU3-A16: U8.16 (IOL_10B)
- net CPU3-A2 is gone; now on net CPU3-A23: U8.7 (IOL_4A)
- net CPU3-A3 is gone; now on net ~{CPU3-LDS}: U8.3 (IOL_3A)
- net CPU3-A4 is gone; now on net ~{CPU3-AS}: U8.1 (IOL_2A)
- net CPU3-A5 is gone; now on net ~{CPU3-UDS}: U8.2 (IOL_2B)
- net CPU3-A6 is gone; now on net CPU3-R/~{W}: U8.4 (IOL_3B)
- net CPU3-A7 is gone; now on net CPU3-A22: U8.8 (IOL_4B)
- net CPU3-A8 is gone; now on net CPU3-A20: U8.10 (IOL_5B)
- net CPU3-A9 is gone; now on net CPU3-A19: U8.11 (IOL_8A)
- net CPU3-D0 is gone; now on net VID-HSYNC3: U8.47 (IOB_79)
- net CPU3-D1 is gone; now on net VID-R1: U8.49 (IOB_81_GBIN5)
- net CPU3-D14 is gone; now on net VID-G3: U8.39 (IOB_61)
- net CPU3-D15 is gone; now on net VID-G2: U8.38 (IOB_57)
- net CPU3-D2 is gone; now on net VID-R3: U8.55 (IOB_91)
- net CPU3-D7 is gone; now on net VID-R2: U8.52 (IOB_82_GBIN4)
- net CPU3-D8 is gone; now on net VID-R0: U8.48 (IOB_80)
- net CPU3-D9 is gone; now on net VID-VSYNC3: U8.45 (IOB_73)
- net VRAM-CKE is gone; now on net VRAM-D1: U8.112 (IOT_169)
- net +3V3: now also U12.1 (VDD), U12.14 (VDD), U12.27 (VDD), U12.3 (VDDQ), U12.37 (CKE), U12.43 (VDDQ), U12.49 (VDDQ), U12.9 (VDDQ)
- net +5V: now also U7.10 (IN3_P), U7.9 (IN3_N); no longer U7.5 (IN2_P), U7.6 (IN2_N)
- net AUXSW: no longer U8.91 (IOR_139)
- net CPU3-A16: no longer U8.20 (IOL_13B_GBIN7)
- net CPU3-A17: no longer U8.21 (IOL_14A_GBIN6)
- net CPU3-A18: no longer U8.22 (IOL_14B)
- net CPU3-A19: no longer U8.23 (IOL_17A)
- net CPU3-A20: no longer U8.24 (IOL_17B)
- net CPU3-A21: no longer U8.25 (IOL_18A)
- net CPU3-A22: no longer U8.26 (IOL_18B)
- net CPU3-A23: no longer U8.28 (IOL_23A)
- net CPU3-R/~{W}: no longer U8.29 (IOL_23B)
- net GND: now also R29.1, R52.1, R68.1, U12.12 (VSSQ), U12.19 (~{CS}), U12.28 (VSS), U12.41 (VSS), U12.46 (VSSQ), U12.52 (VSSQ), U12.54 (VSS), U12.6 (VSSQ)
- net MEMSEL0: now also U8.75 (IOR_111); no longer U8.94 (IOR_141_GBIN2)
- net MEMSEL1: now also U8.74 (IOR_110); no longer U8.95 (IOR_144)
- net MEMSEL2: now also U8.73 (IOR_109); no longer U8.96 (IOR_146)
- net VID-B0: now also U8.24 (IOL_17B), R60.1; no longer U8.75 (IOR_111)
- net VID-B1: now also U8.25 (IOL_18A), R59.1; no longer U8.79 (IOR_115)
- net VID-B2: now also U8.26 (IOL_18B), R58.1; no longer U8.73 (IOR_109)
- net VID-B3: now also U8.28 (IOL_23A), R57.1; no longer U8.74 (IOR_110)
- net VID-G0: now also U8.34 (IOL_25B), R44.1; no longer U8.82 (IOR_118)
- net VID-G1: now also U8.37 (IOB_56), R43.1; no longer U8.83 (IOR_119)
- net VID-G2: now also R42.1; no longer U8.80 (IOR_116)
- net VID-G3: now also R41.1; no longer U8.81 (IOR_117)
- net VID-HSYNC3: no longer U8.78 (IOR_114)
- net VID-R0: now also R28.1; no longer U8.87 (IOR_136)
- net VID-R1: now also R27.1; no longer U8.88 (IOR_137)
- net VID-R2: now also R26.1; no longer U8.84 (IOR_120)
- net VID-R3: now also R25.1; no longer U8.85 (IOR_128)
- net VID-VSYNC3: no longer U8.76 (IOR_112)
- net VRAM-A0: now also U8.101 (IOR_160), U12.23 (A0); no longer U8.143 (IOT_221)
- net VRAM-A1: now also U8.102 (IOR_161), U12.24 (A1); no longer U8.138 (IOT_216)
- net VRAM-A10: now also U12.22 (A10); no longer U8.142 (IOT_220)
- net VRAM-A11: now also U8.78 (IOR_114), U12.35 (A11); no longer U8.141 (IOT_219)
- net VRAM-A2: now also U8.104 (IOR_164), U12.25 (A2); no longer U8.139 (IOT_217)
- net VRAM-A3: now also U8.105 (IOR_165), U12.26 (A3); no longer U8.144 (IOT_222)
- net VRAM-A4: now also U8.94 (IOR_141_GBIN2), U12.29 (A4); no longer U8.118 (IOT_177)
- net VRAM-A5: now also U8.95 (IOR_144), U12.30 (A5); no longer U8.117 (IOT_174)
- net VRAM-A6: now also U8.96 (IOR_146), U12.31 (A6); no longer U8.116 (IOT_173)
- net VRAM-A7: now also U8.97 (IOR_147), U12.32 (A7); no longer U8.115 (IOT_172)
- net VRAM-A8: now also U8.98 (IOR_148), U12.33 (A8); no longer U8.114 (IOT_171)
- net VRAM-A9: now also U8.76 (IOR_112), U12.34 (A9); no longer U8.113 (IOT_170)
- net VRAM-CLK: now also U8.80 (IOR_116), U12.38 (CLK); no longer U8.110 (IOT_168)
- net VRAM-D0: now also U8.110 (IOT_168), U12.2 (DQ0); no longer U8.119 (IOT_178)
- net VRAM-D1: now also U12.4 (DQ1); no longer U8.120 (IOT_179)
- net VRAM-D10: now also U8.85 (IOR_128), U12.45 (DQ10); no longer U8.104 (IOR_164)
- net VRAM-D11: now also U8.84 (IOR_120), U12.47 (DQ11); no longer U8.102 (IOR_161)
- net VRAM-D12: now also U8.88 (IOR_137), U12.48 (DQ12); no longer U8.101 (IOR_160)
- net VRAM-D13: now also U8.91 (IOR_139), U12.50 (DQ13); no longer U8.99 (IOR_152)
- net VRAM-D14: now also U8.90 (IOR_138), U12.51 (DQ14); no longer U8.98 (IOR_148)
- net VRAM-D15: now also U8.87 (IOR_136), U12.53 (DQ15); no longer U8.97 (IOR_147)
- net VRAM-D2: now also U8.113 (IOT_170), U12.5 (DQ2); no longer U8.121 (IOT_181)
- net VRAM-D3: now also U8.114 (IOT_171), U12.7 (DQ3); no longer U8.122 (IOT_190)
- net VRAM-D4: now also U8.115 (IOT_172), U12.8 (DQ4); no longer U8.124 (IOT_191)
- net VRAM-D5: now also U8.116 (IOT_173), U12.10 (DQ5); no longer U8.125 (IOT_192)
- net VRAM-D6: now also U8.117 (IOT_174), U12.11 (DQ6); no longer U8.128 (IOT_197_GBIN1)
- net VRAM-D7: now also U8.118 (IOT_177), U12.13 (DQ7); no longer U8.129 (IOT_198_GBIN0)
- net VRAM-D8: now also U8.82 (IOR_118), U12.42 (DQ8); no longer U8.106 (IOR_166)
- net VRAM-D9: now also U8.83 (IOR_119), U12.44 (DQ9); no longer U8.105 (IOR_165)
- net VRAM-LDQM: now also U8.119 (IOT_178), U12.15 (DQML); no longer U8.130 (IOT_206)
- net VRAM-UDQM: now also U8.81 (IOR_117), U12.39 (DQMH); no longer U8.107 (IOR_167)
- net ~{CPU3-AS}: no longer U8.33 (IOL_25A)
- net ~{CPU3-DEN}: now also U8.23 (IOL_17A); no longer U8.37 (IOB_56)
- net ~{CPU3-DTACK}: no longer U8.34 (IOL_25B)
- net ~{CPU3-LDS}: no longer U8.31 (IOL_24A)
- net ~{CPU3-UDS}: no longer U8.32 (IOL_24B)
- net ~{VRAM-CAS}: now also U8.120 (IOT_179), U12.17 (~{CAS}); no longer U8.135 (IOT_213)
- net ~{VRAM-CS}: no longer U8.137 (IOT_215)
- net ~{VRAM-RAS}: now also U8.121 (IOT_181), U12.18 (~{RAS}); no longer U8.136 (IOT_214)
- net ~{VRAM-WE}: now also U8.99 (IOR_152), U12.16 (~{WE}); no longer U8.134 (IOT_212)
- net at R5.2, U7.12 (IN4_P): now also R37.2, R45.2
- net at R4.2, U7.3 (IN1_P): now also R21.2, R30.2
- net at R6.2: now also U7.5 (IN2_P), R53.2, R61.2; no longer U7.10 (IN3_P)
- net at R13.2: now also U7.8 (OUT3); no longer U7.7 (OUT2)
- net CPU3-A13: no longer names the net of U8.18 (IOL_12B)
- net CPU3-A14: no longer names the net of U8.17 (IOL_12A)
- net CPU3-A15: no longer names the net of U8.19 (IOL_13A)
- net CPU3-D10 renamed VID-G7
- net VID-G7: now also R37.1
- net CPU3-D11 renamed VID-G6
- net VID-G6: now also R38.1
- net CPU3-D12 renamed VID-G5
- net VID-G5: now also R39.1
- net CPU3-D13 renamed VID-G4
- net VID-G4: now also R40.1
- net CPU3-D3 renamed VID-R4
- net VID-R4: now also R24.1
- net CPU3-D4 renamed VID-R7
- net VID-R7: now also R21.1
- net CPU3-D5 renamed VID-R6
- net VID-R6: now also R22.1
- net CPU3-D6 renamed VID-R5
- net VID-R5: now also R23.1
- new net: R23.2, R31.1, R32.2
- new net: R39.2, R46.1, R47.2
- new net: R38.2, R45.1, R46.2
- new net: R28.2, R29.2, R36.1
- new net: R27.2, R35.1, R36.2
- new net: R60.2, R67.1, R68.2
- new net: R3.1, U7.6 (IN2_N), U7.7 (OUT2)
- new net: R24.2, R32.1, R33.2
- new net: R59.2, R66.1, R67.2
- new net: R56.2, R63.1, R64.2
- new net: R55.2, R62.1, R63.2
- new net: R58.2, R65.1, R66.2
- new net: R54.2, R61.1, R62.2
- new net: R43.2, R50.1, R51.2
- new net: R42.2, R49.1, R50.2
- new net: R26.2, R34.1, R35.2
- new net: R40.2, R47.1, R48.2
- new net: R22.2, R30.1, R31.2
- new net: R44.2, R51.1, R52.2
- new net: R25.2, R33.1, R34.2
- new net: R41.2, R48.1, R49.2
- new net: R57.2, R64.1, R65.2
- new net CPU3-AD0: U8.144 (IOT_222)
- new net CPU3-AD1: U8.143 (IOT_221)
- new net CPU3-AD10: U8.135 (IOT_213)
- new net CPU3-AD11: U8.134 (IOT_212)
- new net CPU3-AD12: U8.125 (IOT_192)
- new net CPU3-AD13: U8.130 (IOT_206)
- new net CPU3-AD14: U8.129 (IOT_198_GBIN0)
- new net CPU3-AD15: U8.124 (IOT_191)
- new net CPU3-AD2: U8.142 (IOT_220)
- new net CPU3-AD3: U8.141 (IOT_219)
- new net CPU3-AD4: U8.139 (IOT_217)
- new net CPU3-AD5: U8.138 (IOT_216)
- new net CPU3-AD6: U8.137 (IOT_215)
- new net CPU3-AD7: U8.128 (IOT_197_GBIN1)
- new net CPU3-AD8: U8.136 (IOT_214)
- new net CPU3-AD9: U8.122 (IOT_190)
- new net VID-B4: R56.1, U8.29 (IOL_23B)
- new net VID-B5: R55.1, U8.31 (IOL_24A)
- new net VID-B6: R54.1, U8.32 (IOL_24B)
- new net VID-B7: R53.1, U8.33 (IOL_25A)
- new net VRAM-A12: U12.36 (A12), U8.79 (IOR_115)
- new net VRAM-BA0: U12.20 (BA0), U8.107 (IOR_167)
- new net VRAM-BA1: U12.21 (BA1), U8.106 (IOR_166)
Other:
- sheet Mac Interface ports: added CPU-AD[15..0], CPU3-A[23..16], ~{CPU3-AEN}; removed CPU3-A[23..0], CPU3-D[15..0], ~{CPU3-RESET}
- moved on the sheet: C17, C26, C27, C28, C34, J3, R1, R13, R14, R15, R16, R17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

Commit message: Cleanup for DRC
Parts:
- added S1, S2, S3, S4, S5, S6: Conn_01x01, Connector_PinHeader_2.54mm:PinHeader_1x01_P2.54mm_Vertical, symbol Connector_Generic:Conn_01x01
Connections:
- net AUXSW: now also S6.1 (Pin_1)
- net CBSEL0: now also S1.1 (Pin_1)
- net CBSEL1: now also S2.1 (Pin_1)
- net MEMSEL0: now also S3.1 (Pin_1)
- net MEMSEL1: now also S4.1 (Pin_1)
- net MEMSEL2: now also S5.1 (Pin_1)
Other:
- note added: "Configuration Alt Jumpers"
- note added: "Configuration DIP Switches"
- moved on the sheet: C26, C27, C28, C34, R14, R15, R16, R17, R18, R19, SW1
